Commit message: modified robot model

File: patin_description/urdf/astra.urdf.xacro (robot description, xacro)
@@ -5,9 +5,9 @@
       <xacro:insert_block name="joint_origin"/>
       <parent link="${parent}"/>
-      <child link="astra"/>
+      <child link="camera_link"/>
     </joint>
-    <link name="astra">
+    <link name="camera_link">
       <visual>
-        <origin xyz="0 0 0" rpy="0 0 0" />
+        <origin xyz="0 0 0" rpy="0 0 -1.57" />
         <geometry>
           <mesh filename="package://patin_description/model/astra.dae"/>

File: patin_description/urdf/patin.urdf.xacro (robot description, xacro)
@@ -35,5 +35,5 @@
   </xacro:lidar>
   <xacro:astra parent="base_link">
-    <origin xyz="0.1 0.0 0.12" rpy="2.9 0.0 1.57" />
+    <origin xyz="0.1 0.0 0.12" rpy="0.0 -0.24 0.0" />
   </xacro:astra>
 </robot>
